File: Tarea 4/USB SD CARD/USB SD CARD.kicad_pcb (KiCad board)
At the start: 2 copper layers, 22 parts, among them U1 USBLC6-2P6, U2 MT9700-N

Commit message: mi quinto commit
Parts:
- moved R11 25.8 mm to (140.0, 39.2), turned to -90 degrees
- moved R7 21.2 mm to (136.5, 40.0), turned to 180 degrees
- moved R9 18.4 mm to (147.0, 38.5), turned to 90 degrees
- moved R8 14.2 mm to (149.5, 39.5)
- moved R10 12.0 mm to (154.5, 45.5)
- moved R4 7.01 mm to (151.0, 64.5)
- moved R3 4.52 mm to (151.0, 59.5)
- moved U2 3.38 mm to (154.0, 40.5), turned to 90 degrees
- moved R5 3.00 mm to (151.0, 57.0)
- moved R6 0.54 mm to (151.0, 62.0)
- moved C2 0.49 mm to (151.0, 49.5), turned to 180 degrees
Routing:
- net 3.3V: track 41.0 -> 182.9 mm, vias 0 -> 2
- net GND: track 162.3 -> 272.6 mm, vias 0 -> 2
- net idc_SDA: track 0.00 -> 46.0 mm
- net Net-(Card1-DAT1): track 0.00 -> 24.8 mm
- net SPI_MISO: track 0.00 -> 20.2 mm
- net reset: track 0.00 -> 16.5 mm
- net SD_CS: track 0.00 -> 13.1 mm
- net VDD: track 6.55 -> 17.9 mm
- net Net-(Card1-DAT2): track 0.00 -> 10.5 mm
- net Net-(U2-SET): track 14.5 -> 6.79 mm
- net Net-(F2-Pad2): track 26.5 -> 32.1 mm, vias 0 -> 2
- net IM1: track 0.00 -> 3.78 mm
- net IM2: track 0.00 -> 3.70 mm
- net LED: track 0.00 -> 3.13 mm
